File: electronics/pcb_main/power.kicad_sch (KiCad schematic)
At the start: 0 parts

Commit message: Updates
Other:
- company: © 2023 TekLabs Digital Pty Ltd -> © 2023 Teklabs Digital Pty Ltd
Changed lines of the file:
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@@
     (date "2023-05-18")
     (rev "0.2 alpha")
-    (company "© 2023 TekLabs Digital Pty Ltd")
+    (company "© 2023 Teklabs Digital Pty Ltd")
     (comment 1 "Designed by Trevor Attema")
     (comment 2 "MIT License ")
