File: electronics/pcb_main/debug.kicad_sch (KiCad schematic)
At the start: 3 parts, among them J1 SWD Trace, U1 STM32WB55VGY6TR - Seq

Commit message: BOM update
Parts:
- J1: footprint TekLabs:Molex 5035661102 -> (none)
- JP1: footprint TekLabs:MicroJump-Open -> (none)
- U1: footprint TekLabs:STM32WB55VGY6TR -> (none)
Changed lines of the file:
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@@
     (property "Reference" "J1" (id 0) (at 128.27 91.2835 0))
     (property "Value" "SWD Trace" (id 1) (at 128.27 94.0586 0))
-    (property "Footprint" "TekLabs:Molex 5035661102" (id 2) (at 128.27 109.22 0)
+    (property "Footprint" "" (id 2) (at 128.27 109.22 0)
       (effects (font (size 1.27 1.27)) hide)
     )
@@
       (effects (font (size 1.27 1.27)) (justify right))
     )
-    (property "Footprint" "TekLabs:MicroJump-Open" (id 2) (at 151.13 92.71 0)
+    (property "Footprint" "" (id 2) (at 151.13 92.71 0)
       (effects (font (size 1.27 1.27)) hide)
     )
@@
       (effects (font (size 1.524 1.524)) (justify left))
     )
-    (property "Footprint" "TekLabs:STM32WB55VGY6TR" (id 2) (at 181.61 91.44 0)
+    (property "Footprint" "" (id 2) (at 181.61 91.44 0)
       (effects (font (size 1.524 1.524)) hide)
     )
