File: electronics/pcb_main/io.kicad_sch (KiCad schematic)
At the start: 14 parts, among them J2 Touch FFC, M1 Motor_DC, Q1 2N7002, Q2 2N7002, U6 KTD2052

Commit message: Updates
Parts:
- D3: DigiKey 1N4148WL2-TP -> (none); Digikey (none) -> 1N4148WL2-TP
- TP14, TP15: now left out of the parts list
Other:
- company: © 2023 TekLabs Digital Pty Ltd -> © 2023 Teklabs Digital Pty Ltd
Changed lines of the file:
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@@
     (date "2023-05-18")
     (rev "0.2 alpha")
-    (company "© 2023 TekLabs Digital Pty Ltd")
+    (company "© 2023 Teklabs Digital Pty Ltd")
     (comment 1 "Designed by Trevor Attema")
     (comment 2 "MIT License ")
@@
       (effects (font (size 1.27 1.27)) hide)
     )
-    (property "DigiKey" "1N4148WL2-TP" (id 4) (at 167.64 82.55 90)
+    (property "Digikey" "1N4148WL2-TP" (id 5) (at 167.64 82.55 0)
       (effects (font (size 1.27 1.27)) hide)
     )
@@
   )
   (symbol (lib_id "Connector:TestPoint_Probe") (at 220.98 95.25 0) (unit 1)
-    (in_bom yes) (on_board yes) (fields_autoplaced)
+    (in_bom no) (on_board yes) (fields_autoplaced)
     (property "Reference" "TP15" (id 0) (at 224.79 92.754 0)
       (effects (font (size 1.27 1.27)) (justify left))
@@
   )
   (symbol (lib_id "Connector:TestPoint_Probe") (at 161.29 96.52 0) (unit 1)
-    (in_bom yes) (on_board yes) (fields_autoplaced)
+    (in_bom no) (on_board yes) (fields_autoplaced)
     (property "Reference" "TP14" (id 0) (at 165.1 94.024 0)
       (effects (font (size 1.27 1.27)) (justify left))
@@
       (effects (font (size 1.27 1.27)) hide)
     )
-    (property "Vaniman" "" (id 5) (at 226.06 106.68 0)
-      (effects (font (size 1.27 1.27)) hide)
-    )

Commit message: BOM update
Parts:
- BZ1: footprint TekLabs:Transducer TE044003-4 -> (none)
- C32: footprint Capacitor_SMD:C_0603_1608Metric -> (none)
- D1, D2: footprint LED_SMD:LED_LiteOn_LTST-C19HE1WT -> (none)
- D3: footprint Diode_SMD:D_0402_1005Metric -> (none)
- J2: footprint TekLabs:MOLEX_5034800800 -> (none)
- M1: footprint TekLabs:SMT Motor VZ43FM1B8230001L -> (none); Digikey (none) -> 1670-VZ43FM1B8230001LCT-ND
- Q1, Q2: footprint Package_TO_SOT_SMD:SOT-883 -> (none)
- R10, R11: footprint Resistor_SMD:R_0402_1005Metric -> (none); Digikey (none) -> 311-1.00MLRCT-ND
- TP14, TP15: footprint TekLabs:MicroTest-1 -> (none)
- U6: footprint Package_DFN_QFN:DFN-8-1EP_2x2mm_P0.5mm_EP1.05x1.75mm -> (none)
Changed lines of the file:
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@@
       (effects (font (size 1.27 1.27)) (justify left))
     )
-    (property "Footprint" "Package_TO_SOT_SMD:SOT-883" (id 2) (at 240.03 103.505 0)
+    (property "Footprint" "" (id 2) (at 240.03 103.505 0)
       (effects (font (size 1.27 1.27) italic) (justify left) hide)
     )
@@
       (effects (font (size 1.27 1.27)) (justify right))
     )
-    (property "Footprint" "Diode_SMD:D_0402_1005Metric" (id 2) (at 163.195 82.55 0)
+    (property "Footprint" "" (id 2) (at 163.195 82.55 0)
       (effects (font (size 1.27 1.27)) hide)
     )
@@
       (effects (font (size 1.27 1.27)) (justify left))
     )
-    (property "Footprint" "Package_TO_SOT_SMD:SOT-883" (id 2) (at 181.61 103.505 0)
+    (property "Footprint" "" (id 2) (at 181.61 103.505 0)
       (effects (font (size 1.27 1.27) italic) (justify left) hide)
     )
@@
       (effects (font (size 1.27 1.27)) (justify right))
     )
-    (property "Footprint" "LED_SMD:LED_LiteOn_LTST-C19HE1WT" (id 2) (at 125.73 82.55 0)
+    (property "Footprint" "" (id 2) (at 125.73 82.55 0)
       (effects (font (size 1.27 1.27)) hide)
     )
@@
       (effects (font (size 1.27 1.27)) (justify left))
     )
-    (property "Footprint" "TekLabs:MicroTest-1" (id 2) (at 226.06 95.25 0)
+    (property "Footprint" "" (id 2) (at 226.06 95.25 0)
       (effects (font (size 1.27 1.27)) hide)
     )
@@
       (effects (font (size 1.27 1.27)) (justify right))
     )
-    (property "Footprint" "LED_SMD:LED_LiteOn_LTST-C19HE1WT" (id 2) (at 99.06 82.55 0)
+    (property "Footprint" "" (id 2) (at 99.06 82.55 0)
       (effects (font (size 1.27 1.27)) hide)
     )
@@
       (effects (font (size 1.27 1.27)) (justify left))
     )
-    (property "Footprint" "TekLabs:MicroTest-1" (id 2) (at 166.37 96.52 0)
+    (property "Footprint" "" (id 2) (at 166.37 96.52 0)
       (effects (font (size 1.27 1.27)) hide)
     )
@@
     (property "Reference" "U6" (id 0) (at 69.215 79.9043 0))
     (property "Value" "KTD2052" (id 1) (at 69.215 82.6794 0))
-    (property "Footprint" "Package_DFN_QFN:DFN-8-1EP_2x2mm_P0.5mm_EP1.05x1.75mm" (id 2) (at 69.85 116.84 0)
+    (property "Footprint" "" (id 2) (at 69.85 116.84 0)
       (effects (font (size 1.27 1.27)) hide)
     )
@@
       (effects (font (size 1.27 1.27)) (justify right))
     )
-    (property "Footprint" "Resistor_SMD:R_0402_1005Metric" (id 2) (at 226.06 106.68 0)
+    (property "Footprint" "" (id 2) (at 226.06 106.68 0)
       (effects (font (size 1.27 1.27)) hide)
     )
@@
       (effects (font (size 1.27 1.27)) hide)
     )
+    (property "Digikey" "311-1.00MLRCT-ND" (id 5) (at 226.06 106.68 0)
+      (effects (font (size 1.27 1.27)) hide)
+    )
     (pin "1")
     (pin "2")
@@
       (effects (font (size 1.27 1.27)) (justify left))
     )
-    (property "Footprint" "TekLabs:SMT Motor VZ43FM1B8230001L" (id 2) (at 179.07 82.296 0)
+    (property "Footprint" "" (id 2) (at 179.07 82.296 0)
       (effects (font (size 1.27 1.27)) hide)
     )
@@
       (effects (font (size 1.27 1.27)) hide)
     )
+    (property "Digikey" "1670-VZ43FM1B8230001LCT-ND" (id 4) (at 179.07 80.01 0)
+      (effects (font (size 1.27 1.27)) hide)
+    )
     (pin "1")
     (pin "2")
@@
       (effects (font (size 1.27 1.27)) (justify left))
     )
-    (property "Footprint" "TekLabs:Transducer TE044003-4" (id 2) (at 239.395 78.74 90)
+    (property "Footprint" "" (id 2) (at 239.395 78.74 90)
       (effects (font (size 1.27 1.27)) hide)
     )
@@
       (effects (font (size 1.27 1.27)) (justify right))
     )
-    (property "Footprint" "Capacitor_SMD:C_0603_1608Metric" (id 2) (at 57.15 91.44 0)
+    (property "Footprint" "" (id 2) (at 57.15 91.44 0)
       (effects (font (size 1.27 1.27)) hide)
     )
@@
       (effects (font (size 1.27 1.27)) (justify right))
     )
-    (property "Footprint" "Resistor_SMD:R_0402_1005Metric" (id 2) (at 167.64 106.68 0)
+    (property "Footprint" "" (id 2) (at 167.64 106.68 0)
       (effects (font (size 1.27 1.27)) hide)
     )
@@
     )
     (property "Vaniman" "" (id 5) (at 167.64 106.68 0)
+      (effects (font (size 1.27 1.27)) hide)
+    )
+    (property "Digikey" "311-1.00MLRCT-ND" (id 6) (at 167.64 106.68 0)
       (effects (font (size 1.27 1.27)) hide)
     )
@@
       (effects (font (size 1.27 1.27)) (justify left))
     )
-    (property "Footprint" "TekLabs:MOLEX_5034800800" (id 2) (at 116.84 151.13 0)
-      (effects (font (size 1.27 1.27)) hide)
-    )
+    (property "Footprint" "" (id 2) (at 116.84 151.13 0)
+      (effects (font (size 1.27 1.27)) hide)
+    )
