File: electronics/pcb_main/mcu-power.kicad_sch (KiCad schematic)
At the start: 16 parts, among them U1 STM32WB55VGY6TR - Seq

Commit message: Updates
Parts:
- TP6, TP7, TP8: now left out of the parts list
Other:
- company: © 2023 TekLabs Digital Pty Ltd -> © 2023 Teklabs Digital Pty Ltd
Changed lines of the file:
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@@
     (date "2023-05-18")
     (rev "0.2 alpha")
-    (company "© 2023 TekLabs Digital Pty Ltd")
+    (company "© 2023 Teklabs Digital Pty Ltd")
     (comment 1 "Designed by Trevor Attema")
     (comment 2 "MIT License ")
@@
   )
   (symbol (lib_id "Connector:TestPoint_Probe") (at 59.69 74.93 0) (unit 1)
-    (in_bom yes) (on_board yes)
+    (in_bom no) (on_board yes)
     (property "Reference" "TP6" (id 0) (at 63.5 72.434 0)
       (effects (font (size 1.27 1.27)) (justify left))
@@
   )
   (symbol (lib_id "Connector:TestPoint_Probe") (at 88.9 77.47 0) (unit 1)
-    (in_bom yes) (on_board yes) (fields_autoplaced)
+    (in_bom no) (on_board yes) (fields_autoplaced)
     (property "Reference" "TP7" (id 0) (at 92.71 74.974 0)
       (effects (font (size 1.27 1.27)) (justify left))
@@
   )
   (symbol (lib_id "Connector:TestPoint_Probe") (at 81.28 95.25 0) (mirror y) (unit 1)
-    (in_bom yes) (on_board yes) (fields_autoplaced)
+    (in_bom no) (on_board yes) (fields_autoplaced)
     (property "Reference" "TP8" (id 0) (at 81.915 92.754 0)
       (effects (font (size 1.27 1.27)) (justify right))

Commit message: BOM update
Parts:
- C10, C11, C12, C13, C14, C15, C7, C8, C9: footprint Capacitor_SMD:C_0402_1005Metric -> (none)
- C6: footprint Capacitor_SMD:C_0603_1608Metric -> (none)
- L1, L2: footprint Inductor_SMD:L_0603_1608Metric -> (none)
- TP6, TP7, TP8: footprint TekLabs:MicroTest-1 -> (none)
- U1: footprint TekLabs:STM32WB55VGY6TR -> (none)
Changed lines of the file:
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@@
       (effects (font (size 1.27 1.27)) (justify left))
     )
-    (property "Footprint" "Capacitor_SMD:C_0402_1005Metric" (id 2) (at 133.35 146.05 0)
+    (property "Footprint" "" (id 2) (at 133.35 146.05 0)
       (effects (font (size 1.27 1.27)) hide)
     )
@@
       (effects (font (size 1.27 1.27)) (justify left))
     )
-    (property "Footprint" "Capacitor_SMD:C_0402_1005Metric" (id 2) (at 59.69 90.17 0)
+    (property "Footprint" "" (id 2) (at 59.69 90.17 0)
       (effects (font (size 1.27 1.27)) hide)
     )
@@
       (effects (font (size 1.27 1.27)) (justify left))
     )
-    (property "Footprint" "Capacitor_SMD:C_0402_1005Metric" (id 2) (at 182.88 146.05 0)
+    (property "Footprint" "" (id 2) (at 182.88 146.05 0)
       (effects (font (size 1.27 1.27)) hide)
     )
@@
     (property "Reference" "L2" (id 0) (at 78.74 87.0925 90))
     (property "Value" "10nH" (id 1) (at 78.74 89.8676 90))
-    (property "Footprint" "Inductor_SMD:L_0603_1608Metric" (id 2) (at 78.74 91.44 0)
+    (property "Footprint" "" (id 2) (at 78.74 91.44 0)
       (effects (font (size 1.27 1.27)) hide)
     )
@@
       (effects (font (size 1.27 1.27)) (justify left))
     )
-    (property "Footprint" "Capacitor_SMD:C_0402_1005Metric" (id 2) (at 152.4 146.05 0)
+    (property "Footprint" "" (id 2) (at 152.4 146.05 0)
       (effects (font (size 1.27 1.27)) hide)
     )
@@
       (effects (font (size 1.27 1.27)) (justify left))
     )
-    (property "Footprint" "Capacitor_SMD:C_0402_1005Metric" (id 2) (at 172.72 146.05 0)
+    (property "Footprint" "" (id 2) (at 172.72 146.05 0)
       (effects (font (size 1.27 1.27)) hide)
     )
@@
       (effects (font (size 1.27 1.27)) (justify right))
     )
-    (property "Footprint" "Inductor_SMD:L_0603_1608Metric" (id 2) (at 72.39 95.25 0)
+    (property "Footprint" "" (id 2) (at 72.39 95.25 0)
       (effects (font (size 1.27 1.27)) hide)
     )
@@
       (effects (font (size 1.27 1.27)) (justify left))
     )
-    (property "Footprint" "Capacitor_SMD:C_0402_1005Metric" (id 2) (at 72.39 104.14 0)
+    (property "Footprint" "" (id 2) (at 72.39 104.14 0)
       (effects (font (size 1.27 1.27)) hide)
     )
@@
       (effects (font (size 1.27 1.27)) (justify left))
     )
-    (property "Footprint" "TekLabs:MicroTest-1" (id 2) (at 64.77 74.93 0)
+    (property "Footprint" "" (id 2) (at 64.77 74.93 0)
       (effects (font (size 1.27 1.27)) hide)
     )
@@
       (effects (font (size 1.27 1.27)) (justify left))
     )
-    (property "Footprint" "Capacitor_SMD:C_0603_1608Metric" (id 2) (at 50.8 90.17 0)
+    (property "Footprint" "" (id 2) (at 50.8 90.17 0)
       (effects (font (size 1.27 1.27)) hide)
     )
@@
       (effects (font (size 1.27 1.27)) (justify left))
     )
-    (property "Footprint" "Capacitor_SMD:C_0402_1005Metric" (id 2) (at 142.24 146.05 0)
+    (property "Footprint" "" (id 2) (at 142.24 146.05 0)
       (effects (font (size 1.27 1.27)) hide)
     )
@@
       (effects (font (size 1.524 1.524)) (justify left))
     )
-    (property "Footprint" "TekLabs:STM32WB55VGY6TR" (id 2) (at 110.49 77.47 0)
+    (property "Footprint" "" (id 2) (at 110.49 77.47 0)
       (effects (font (size 1.524 1.524)) hide)
     )
@@
       (effects (font (size 1.27 1.27)) (justify left))
     )
-    (property "Footprint" "TekLabs:MicroTest-1" (id 2) (at 93.98 77.47 0)
+    (property "Footprint" "" (id 2) (at 93.98 77.47 0)
       (effects (font (size 1.27 1.27)) hide)
     )
@@
       (effects (font (size 1.524 1.524)))
     )
-    (property "Footprint" "TekLabs:STM32WB55VGY6TR" (id 2) (at 198.12 63.5 0)
+    (property "Footprint" "" (id 2) (at 198.12 63.5 0)
       (effects (font (size 1.524 1.524)) hide)
     )
@@
       (effects (font (size 1.27 1.27)) (justify right))
     )
-    (property "Footprint" "TekLabs:MicroTest-1" (id 2) (at 76.2 95.25 0)
+    (property "Footprint" "" (id 2) (at 76.2 95.25 0)
       (effects (font (size 1.27 1.27)) hide)
     )
@@
       (effects (font (size 1.27 1.27)) (justify left))
     )
-    (property "Footprint" "Capacitor_SMD:C_0402_1005Metric" (id 2) (at 162.56 146.05 0)
+    (property "Footprint" "" (id 2) (at 162.56 146.05 0)
       (effects (font (size 1.27 1.27)) hide)
     )
@@
       (effects (font (size 1.27 1.27)) (justify left))
     )
-    (property "Footprint" "Capacitor_SMD:C_0402_1005Metric" (id 2) (at 123.19 146.05 0)
-      (effects (font (size 1.27 1.27)) hide)
-    )
+    (property "Footprint" "" (id 2) (at 123.19 146.05 0)
+      (effects (font (size 1.27 1.27)) hide)
+    )
