File: electronics/pcb_main/mcu.kicad_sch (KiCad schematic)
At the start: 26 parts, among them SW1 RESET, U1 STM32WB55VGY6TR - Seq, U3 MLPF-WB55-01E3, Y1 32MHz, Y2 32768kHz

Commit message: Updates
Parts:
- TP1, TP2, TP3, TP4, TP5: now left out of the parts list
Other:
- company: © 2023 TekLabs Digital Pty Ltd -> © 2023 Teklabs Digital Pty Ltd
Changed lines of the file:
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@@
     (date "2023-05-18")
     (rev "0.2 alpha")
-    (company "© 2023 TekLabs Digital Pty Ltd")
+    (company "© 2023 Teklabs Digital Pty Ltd")
     (comment 1 "Designed by Trevor Attema")
     (comment 2 "MIT License ")
@@
   )
   (symbol (lib_id "Connector:TestPoint_Probe") (at 251.46 133.35 0) (unit 1)
-    (in_bom yes) (on_board yes) (fields_autoplaced)
+    (in_bom no) (on_board yes) (fields_autoplaced)
     (property "Reference" "TP2" (id 0) (at 255.27 130.854 0)
       (effects (font (size 1.27 1.27)) (justify left))
@@
   )
   (symbol (lib_id "Connector:TestPoint_Probe") (at 125.73 60.96 0) (unit 1)
-    (in_bom yes) (on_board yes) (fields_autoplaced)
+    (in_bom no) (on_board yes) (fields_autoplaced)
     (property "Reference" "TP4" (id 0) (at 129.54 58.464 0)
       (effects (font (size 1.27 1.27)) (justify left))
@@
   )
   (symbol (lib_id "Connector:TestPoint_Probe") (at 142.24 147.32 0) (unit 1)
-    (in_bom yes) (on_board yes) (fields_autoplaced)
+    (in_bom no) (on_board yes) (fields_autoplaced)
     (property "Reference" "TP5" (id 0) (at 146.05 144.824 0)
       (effects (font (size 1.27 1.27)) (justify left))
@@
   )
   (symbol (lib_id "Connector:TestPoint_Probe") (at 39.37 138.43 0) (unit 1)
-    (in_bom yes) (on_board yes) (fields_autoplaced)
+    (in_bom no) (on_board yes) (fields_autoplaced)
     (property "Reference" "TP1" (id 0) (at 43.18 135.934 0)
       (effects (font (size 1.27 1.27)) (justify left))
@@
   )
   (symbol (lib_id "Connector:TestPoint_Probe") (at 125.73 55.88 0) (unit 1)
-    (in_bom yes) (on_board yes) (fields_autoplaced)
+    (in_bom no) (on_board yes) (fields_autoplaced)
     (property "Reference" "TP3" (id 0) (at 129.54 53.384 0)
       (effects (font (size 1.27 1.27)) (justify left))

Commit message: BOM update
Parts:
- AE1: footprint TekLabs:Johanson_2450AT43B100E -> (none)
- BOOT0: footprint TekLabs:MicroJump -> (none)
- C1, C2, C3, C4, C5: footprint Capacitor_SMD:C_0402_1005Metric -> (none)
- C34: footprint Capacitor_SMD:C_0402_1005Metric -> (none); Digikey (none) -> EMK105BJ105KV-F
- C35: footprint Capacitor_SMD:C_0402_1005Metric -> (none); Digikey (none) -> GRM155R71H473ME14D
- R1, R12, R13, R14, R15, R2: footprint Resistor_SMD:R_0402_1005Metric -> (none); Digikey (none) -> 1292-WR04X1001FTLCT-ND
- R3: footprint Resistor_SMD:R_0402_1005Metric -> (none); Digikey (none) -> 311-47.0KLRCT-ND
- SW1: footprint Button_Switch_SMD:SW_SPST_B3U-1100P -> (none)
- TP1, TP2, TP3, TP4, TP5: footprint TekLabs:MicroTest-1 -> (none)
- U1: footprint TekLabs:STM32WB55VGY6TR -> (none)
- U3: footprint TekLabs:MLPF-WB55-01E3 -> (none)
- Y1: footprint Crystal:Crystal_SMD_EuroQuartz_X22-4Pin_2.5x2.0mm -> (none); Digikey 830107820709 -> 1923-830107820709CT-ND
- Y2: footprint Crystal:Crystal_SMD_MicroCrystal_CM9V-T1A-2Pin_1.6x1.0mm -> (none); Digikey CM9V-T1A-32.768KHZ-7PF-100PPM-TA-QC -> 2195-CM9V-T1A-32.768KHZ-7PF-100PPM-TA-QCCT-ND
