File: electronics/pcb_main/sensors.kicad_sch (KiCad schematic)
At the start: 2 parts, among them U7 LSM6DSV16XTR

Commit message: Updates
Other:
- company: © 2023 TekLabs Digital Pty Ltd -> © 2023 Teklabs Digital Pty Ltd
Changed lines of the file:
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@@
     (date "2023-05-18")
     (rev "0.2 alpha")
-    (company "© 2023 TekLabs Digital Pty Ltd")
+    (company "© 2023 Teklabs Digital Pty Ltd")
     (comment 1 "Designed by Trevor Attema")
     (comment 2 "MIT License ")

Commit message: BOM update
Parts:
- C33: footprint Capacitor_SMD:C_0603_1608Metric -> (none)
- U7: footprint TekLabs:LSM6DSV16XTR -> (none)
Changed lines of the file:
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@@
       (effects (font (size 1.524 1.524)))
     )
-    (property "Footprint" "TekLabs:LSM6DSV16XTR" (id 2) (at 154.94 85.344 0)
+    (property "Footprint" "" (id 2) (at 154.94 85.344 0)
       (effects (font (size 1.524 1.524)) hide)
     )
@@
       (effects (font (size 1.27 1.27)) (justify right))
     )
-    (property "Footprint" "Capacitor_SMD:C_0603_1608Metric" (id 2) (at 119.38 130.81 0)
+    (property "Footprint" "" (id 2) (at 119.38 130.81 0)
       (effects (font (size 1.27 1.27)) hide)
     )
