File: electronics/pcb_main/tektag.kicad_pcb (KiCad board)
At the start: 6 copper layers, 26 x 25 mm, 93 parts, among them J1 SWD Trace, J2 Touch FFC, J3 ExtBatt, M1 Motor_DC, Q1 2N7002, Q2 2N7002, U1 STM32WB55VGY6TR - Seq, U3 MLPF-WB55-01E3, U4 BQ51052BYFP, U5 TLV75533PDRV, U6 KTD2052, U7 LSM6DSV16XTR, Y1 32MHz, Y2 32768kHz

Commit message: Updates
Parts:
- J1: footprint TekLabs:MOLEX_5035481220 -> TekLabs:Molex 5035661102
- moved J1 1.64 mm to (128.8, 95.2), turned to 90 degrees
Connections:
- J1 pad 10: /MCU/Debug/TRACED2 -> /MCU/Debug/TRACED3
- J1 pad 2: /MCU/Debug/SWCLK -> Net-(JP1-Pad1)
- J1 pad 3: Net-(J1-Pad3) -> /MCU/~{nRESET}
- J1 pad 4: /MCU/Debug/TRACECLK -> /MCU/Debug/SWDIO
- J1 pad 5: /MCU/Debug/SWDIO -> /MCU/Debug/SWCLK
- J1 pad 6: /MCU/Debug/TRACED0 -> /MCU/Debug/TRACECLK
- J1 pad 7: /MCU/~{nRESET} -> /MCU/Debug/TRACED0
- J1 pad 9: GND -> /MCU/Debug/TRACED2
- JP1 pad 1: Net-(J1-Pad3) -> Net-(JP1-Pad1)
Routing:
- net Net-(J1-Pad3): track 22.0 -> 0.00 mm, vias 2 -> 0
- net Net-(JP1-Pad1): track 0.00 -> 16.4 mm, vias 0 -> 2
- net /MCU/Debug/TRACED3: track 11.1 -> 4.36 mm, vias 3 -> 1
- net /MCU/Debug/TRACED1: track 11.6 -> 6.22 mm, vias 3 -> 2
- net VDD: track 53.6 -> 58.0 mm, vias 24 -> 23
- net /MCU/Debug/TRACED2: track 12.0 -> 7.86 mm, vias 3 -> 1
- net /MCU/Debug/TRACECLK: track 8.47 -> 5.45 mm, vias 3 -> 1
- net GND: track 21.7 -> 24.4 mm, vias 59 -> 58
- net /MCU/Debug/SWDIO: track 10.1 -> 7.82 mm, vias 3 -> 1
- net /MCU/~{nRESET}: track 12.4 -> 14.6 mm
- net Net-(TH1-Pad1): track 14.0 -> 16.1 mm
- net /MCU/Debug/TRACED0: track 8.87 -> 6.86 mm, vias 3 -> 1
- net /LED - Haptic - Buzzer - Touch/BUZZER_EN: track 20.1 -> 22.0 mm
- net Net-(R15-Pad1): track 16.8 -> 15.1 mm
- net Net-(C1-Pad2): track 7.11 -> 5.90 mm
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- added copper zone on B.Cu, net GND
Other:
- board text added: "Introducing Teklabs Digital's latest open-source marvel. A sophisticated, state-of-the-art BioSensor design for IoT devices. This community project, released under the MIT License, showcases our commitment to pushing the boundaries of digital design innovation. We are passionate about blending technology and creativity to produce designs that power the future of IoT. Our team can design your devi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"
- board text added: "TekTag BioSensor PCB"
- board text added: "Use Cases - Contactless cardiac monitoring via Ballistocardiology (BCG) - Pressure area management - bed turn and movement detection - Fall detection - Dementia geo-fence alerting - Respiratory monitoring - Sleep pattern monitoring"

Commit message: BOM update
Routing:
- net /LED - Haptic - Buzzer - Touch/I2C.SDA: track 20.2 -> 30.4 mm
- net GND: track 24.4 -> 23.2 mm, vias 58 -> 59
- net /MCU/Debug/SWDIO: track 7.82 -> 8.89 mm
- net Net-(R15-Pad1): track 15.1 -> 16.1 mm
- net /LED - Haptic - Buzzer - Touch/I2C.SCL: track 21.7 -> 22.5 mm
- net /MCU/Debug/TRACECLK: track 5.45 -> 4.86 mm
- net /MCU/~{nRESET}: track 14.6 -> 15.1 mm
- added copper zone on B.Cu, net (none)
- added copper zone on F.Cu, net (none)
- removed copper zone on B.Cu, net GND
