File: electronics/pcb_main/tektag.kicad_sch (KiCad schematic)
At the start: 0 parts

Commit message: Updates
Other:
- note added: "Introducing Teklabs Digital's latest open-source marvel. A sophisticated, state-of-the-art BioSensor design for IoT devices. This community project, released under the MIT License, showcases our commitment to pushing the boundaries of digital design innovation. We are passionate about blending technology and creativity to produce designs that power the future of IoT. Our team can design your devi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"
- company: © 2023 TekLabs Digital Pty Ltd -> © 2023 Teklabs Digital Pty Ltd
