File: electronics/pcb_main/wcharge.kicad_sch (KiCad schematic)
At the start: 35 parts, among them J3 ExtBatt, U4 BQ51052BYFP, U5 TLV75533PDRV

Commit message: Updates
Parts:
- TP10, TP11, TP12, TP13, TP9: now left out of the parts list
Other:
- company: © 2023 TekLabs Digital Pty Ltd -> © 2023 Teklabs Digital Pty Ltd
Changed lines of the file:
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@@
     (date "2023-05-18")
     (rev "0.2 alpha")
-    (company "© 2023 TekLabs Digital Pty Ltd")
+    (company "© 2023 Teklabs Digital Pty Ltd")
     (comment 1 "Designed by Trevor Attema")
     (comment 2 "MIT License ")
@@
   )
   (symbol (lib_id "Connector:TestPoint_Probe") (at 229.87 82.55 0) (unit 1)
-    (in_bom yes) (on_board yes) (fields_autoplaced)
+    (in_bom no) (on_board yes) (fields_autoplaced)
     (property "Reference" "TP13" (id 0) (at 233.68 80.054 0)
       (effects (font (size 1.27 1.27)) (justify left))
@@
   )
   (symbol (lib_id "Connector:TestPoint_Probe") (at 124.46 83.82 0) (unit 1)
-    (in_bom yes) (on_board yes) (fields_autoplaced)
+    (in_bom no) (on_board yes) (fields_autoplaced)
     (property "Reference" "TP9" (id 0) (at 128.27 81.324 0)
       (effects (font (size 1.27 1.27)) (justify left))
@@
   )
   (symbol (lib_id "Connector:TestPoint_Probe") (at 190.5 82.55 0) (unit 1)
-    (in_bom yes) (on_board yes)
+    (in_bom no) (on_board yes)
     (property "Reference" "TP12" (id 0) (at 194.31 81.28 0)
       (effects (font (size 1.27 1.27)) (justify left))
@@
   )
   (symbol (lib_id "Connector:TestPoint_Probe") (at 138.43 114.3 0) (unit 1)
-    (in_bom yes) (on_board yes) (fields_autoplaced)
+    (in_bom no) (on_board yes) (fields_autoplaced)
     (property "Reference" "TP11" (id 0) (at 142.24 111.804 0)
       (effects (font (size 1.27 1.27)) (justify left))
@@
   )
   (symbol (lib_id "Connector:TestPoint_Probe") (at 142.24 83.82 0) (unit 1)
-    (in_bom yes) (on_board yes) (fields_autoplaced)
+    (in_bom no) (on_board yes) (fields_autoplaced)
     (property "Reference" "TP10" (id 0) (at 146.05 81.324 0)
       (effects (font (size 1.27 1.27)) (justify left))

Commit message: BOM update
Parts:
- BT1: footprint TekLabs:CP1254 Battery -> (none)
- C16, C17, C18, C19, C20, C21, C22, C23, C24, C25, C26, C27: footprint Capacitor_SMD:C_0402_1005Metric -> (none)
- C28, C29: footprint Capacitor_SMD:C_0402_1005Metric -> (none); Digikey GRM188R6YA106MA73D -> (none)
- C30, C31: footprint Capacitor_SMD:C_0603_1608Metric -> (none)
- J3, L3: footprint Connector_PinHeader_1.27mm:PinHeader_1x02_P1.27mm_Vertical -> (none)
- JP2: footprint TekLabs:MicroJump -> (none)
- R16: footprint Resistor_SMD:R_0402_1005Metric -> (none); Digikey (none) -> YAG5650CT-ND
- R4: footprint Resistor_SMD:R_0402_1005Metric -> (none); Digikey (none) -> 311-2.40KLRCT-ND
- R5: footprint Resistor_SMD:R_0402_1005Metric -> (none); Digikey (none) -> 311-100KLRCT-ND
- R6: footprint Resistor_SMD:R_0402_1005Metric -> (none); Digikey (none) -> 311-820LRCT-ND
- R7: footprint Resistor_SMD:R_0402_1005Metric -> (none); Digikey (none) -> 311-220LRCT-ND
- R8: footprint Resistor_SMD:R_0402_1005Metric -> (none); Digikey (none) -> 311-47.0KLRCT-ND
- R9: footprint Resistor_SMD:R_0402_1005Metric -> (none); Digikey (none) -> 311-3.30MLRCT-ND
- TH1: footprint Resistor_SMD:R_0402_1005Metric -> (none)
- TP10, TP11, TP12, TP13, TP9: footprint TekLabs:MicroTest-1 -> (none)
- U4: footprint Package_BGA:Texas_DSBGA-28_1.9x3.0mm_Layout4x7_P0.4mm -> (none)
- U5: footprint Package_SON:WSON-6-1EP_2x2mm_P0.65mm_EP1x1.6mm -> (none)
